File: fuji-mini-v2/fuji-mini-v2.kicad_sch (KiCad schematic)
At the start: 0 parts

Commit message: Schematic Assembly
Parts:
- added BCKWRD/FRWD1, PLAY/PAUSE1: SW_Push, symbol Switch:SW_Push
- added BT1: Battery_Cell, symbol Device:Battery_Cell
- added C1, C10, C11, C16, C17, C2, C3, C4, C5, C6, C7, C8, C9: 100nF, symbol Device:C
- added C12, C13, C14, C15, C20: 1uF, symbol Device:C
- added C18, C19: 220uF, symbol Device:C_Polarized
- added C21, C22, C23: 10uF, symbol Device:C
- added D1: LED, symbol Device:LED
- added J1: Micro_SD_Card, symbol Connector:Micro_SD_Card
- added J2: AudioJack3_SwitchT, symbol Connector_Audio:AudioJack3_SwitchT
- added J3: USB_C_Receptacle, symbol Connector:USB_C_Receptacle
- added R1, R12, R13, R14, R15, R17, R2, R20, R3, R4, R9: 10k, symbol Device:R
- added R10, R11: 4.7kF, symbol Device:R
- added R16: 2k, symbol Device:R
- added R18, R19: 5.1k, symbol Device:R
- added R21: 1k, symbol Device:R
- added R5, R6, R7, R8: 20k, symbol Device:R
- added SW1: RotaryEncoder_Switch, symbol Device:RotaryEncoder_Switch
- added U1: ESP32-S3, Package_DFN_QFN:QFN-56-1EP_7x7mm_P0.4mm_EP4x4mm, symbol MCU_Espressif:ESP32-S3
- added U2: PCM5102A, Package_SO:TSSOP-20_4.4x6.5mm_P0.65mm, symbol Audio:PCM5102A
- added U3: TPA6110A2DGN, Package_SO:HVSSOP-8-1EP_3x3mm_P0.65mm_EP1.57x1.89mm, symbol Amplifier_Audio:TPA6110A2DGN
- added U4: ER_OLEDM0.91_1x-I2C, Display:ER_OLEDM0.91_1x-I2C, symbol Display_Graphic:ER_OLEDM0.91_1x-I2C
- added U5: MCP73831-2-MC, Package_DFN_QFN:DFN-8-1EP_3x2mm_P0.5mm_EP1.7x1.4mm, symbol Battery_Management:MCP73831-2-MC
- added U6: AMS1117-3.3, Package_TO_SOT_SMD:SOT-223-3_TabPin2, symbol Regulator_Linear:AMS1117-3.3
Connections:
- new net: C15.1, U2.7 (OUTR)
- new net: C1.2, J1.4 (VDD)
- new net: C12.1, U2.2 (CAPP)
- new net: C12.2, U2.4 (CAPM)
- new net: J3.A5 (CC1), R18.2
- new net: R5.2, R6.2, U3.4 (IN2-)
- new net: R16.2, U5.8 (PROG)
- new net: R7.2, R8.2, U3.8 (IN1-)
- new net: R21.1, U5.5 (STAT)
- new net: D1.1 (K), R21.2
- new net: R3.1, U1.4 (CHIP_PU)
- new net: C17.1, U2.5 (VNEG)
- new net: C13.1, U3.1 (BYPASS)
- new net: J1.1 (DAT2), R1.2
- new net: J3.B5 (CC2), R19.2
- new net: C14.1, U2.6 (OUTL)
- new net: C16.1, U2.18 (LDOO)
- new net: R17.1, SW1.S2
- new net: J1.8 (DAT1), R2.2
- new net +3V3: BCKWRD/FRWD1.1, BT1.2 (-), C1.1, C10.1, C10.2, C11.1, C11.2, C13.2, C16.2, C17.2, C2.1, C2.2, C20.1, C21.1, C22.1, C22.2, C23.2, C3.1, C3.2, C4.1, C4.2, C5.1, C5.2, C6.1, C6.2, C7.1, C7.2, C8.1, C8.2, C9.1, C9.2, D1.2 (A), J1.6 (VSS), J1.SH (SHIELD), J2.S, J3.A1 (GND), J3.A12 (GND), J3.B1 (GND), J3.B12 (GND), J3.SH (SHIELD), PLAY/PAUSE1.1, R1.1, R10.2, R11.1, R12.1, R13.1, R14.2, R15.1, R16.1, R17.2, R18.1, R19.1, R2.1, R20.1, R3.2, R4.2, R9.1, SW1.C, SW1.S1, U1.2 (VDD3P3), U1.20 (VDD3P3_RTC), U1.29 (VDD_SPI), U1.3 (VDD3P3), U1.46 (VDD3P3_CPU), U1.55 (VDDA), U1.56 (VDDA), U1.57 (GND), U2.1 (CPVDD), U2.10 (DEMP), U2.11 (FLT), U2.16 (FMT), U2.19 (DGND), U2.20 (DVDD), U2.3 (CPGND), U2.8 (AVDD), U2.9 (AGND), U3.2 (GND), U3.6 (VDD), U3.9 (GND), U4.1 (GND), U4.2 (VCC), U5.6 (V_{SS}), U6.1 (GND), U6.2 (VO)
- new net AMP_ENABLE: R9.2, U1.23 (GPIO17), U3.3 (SHDN)
- new net BTN_NEXT: BCKWRD/FRWD1.2, R20.2
- new net BTN_PLAY: PLAY/PAUSE1.2, R14.1
- new net DAC_MUTE: R4.1, U1.19 (GPIO14), U2.17 (XSMT)
- new net DAC_OUTL: C14.2, R7.1
- new net DAC_OUTR: C15.2, R5.1
- new net ENC_A: R12.2, SW1.A
- new net ENC_B: R13.2, SW1.B
- new net GPIO10: J1.2 (DAT3/CD), U1.15 (GPIO10)
- new net GPIO11: J1.3 (CMD), U1.16 (GPIO11)
- new net GPIO12: J1.5 (CLK), U1.17 (GPIO12)
- new net GPIO13: J1.7 (DAT0), U1.18 (GPIO13)
- new net HP_DETECT: J2.TN, R15.2
- new net HP_L: C18.2, J2.T
- new net HP_R: C19.2, J2.R
- new net I2C_SCL: R10.1, U1.13 (GPIO8), U4.3 (SCL)
- new net I2C_SDA: R11.2, U1.14 (GPIO9), U4.4 (SDA)
- new net I2S_BCK: U1.10 (GPIO5), U2.13 (BCK)
- new net I2S_DIN: U1.11 (GPIO6), U2.14 (DIN)
- new net I2S_LRCK: U1.9 (GPIO4), U2.15 (LRCK)
- new net I2S_SCK: U1.12 (GPIO7), U2.12 (SCK)
- new net USB_DN: J3.A7 (D-), U1.25 (GPIO19/USB_D-)
- new net USB_DP: J3.A6 (D+), U1.26 (GPIO20/USB_D+)
- new net VBAT: BT1.1 (+), C21.2, C23.1, U5.3 (V_{BAT}), U5.4 (V_{BAT}), U6.3 (VI)
- new net VDD: C20.2, J3.A4 (VBUS), J3.A9 (VBUS), J3.B4 (VBUS), J3.B9 (VBUS), U5.1 (V_{DD}), U5.2 (V_{DD})
- new net VO1: C18.1, R8.1, U3.7 (VO1)
- new net VO2: C19.1, R6.1, U3.5 (VO2)
- no-connect marks 0 -> 13
Other:
- note added: "AMP (U3)"
- note added: "Battery (U4)"
- note added: "Charger (J3)"
- note added: "DAC (U1)"
- note added: "ESP32"
- note added: "Headphone Jack"
- note added: "OLED (U5)"
- note added: "Regulator (U6)"
- note added: "Rotary + Buttons"
- note added: "SD Card Module"
