File: fuji-mini-v2/fuji-mini-v2.kicad_sch (KiCad schematic)
At the start: 58 parts, among them J1 Micro_SD_Card, J2 AudioJack3_SwitchT, J4 USB_C_Receptacle_USB2.0_14P, SW1 RotaryEncoder_Switch, U1 ESP32-S3, U2 PCM5102A, U3 TPA6110A2DGN, U4 ER_OLEDM0.91_1x-I2C, U5 MCP73831-2-MC, U6 AMS1117-3.3

Commit message: v2.0 2.0 Whole Remake
Parts:
- removed C10, C6, C8: 100nF, Capacitor_SMD:C_0805_2012Metric, symbol Device:C
- removed C23: 10uF, Capacitor_SMD:C_0805_2012Metric, symbol Device:C
- removed R15: 10k, Resistor_SMD:R_0805_2012Metric, symbol Device:R
- removed U1: ESP32-S3, Package_DFN_QFN:QFN-56-1EP_7x7mm_P0.4mm_EP4x4mm, symbol MCU_Espressif:ESP32-S3
- removed U6: AMS1117-3.3, Package_TO_SOT_SMD:SOT-223-3_TabPin2, symbol Regulator_Linear:AMS1117-3.3
- added C21: 1uF, Capacitor_SMD:C_0805_2012Metric, symbol Device:C
- added C7, C9: 100nF, Capacitor_SMD:C_0805_2012Metric, symbol Device:C
- added R2, R4, R6: 10k, Resistor_SMD:R_0805_2012Metric, symbol Device:R
- added SW1, SW2: SW_Push, Button_Switch_THT:SW_PUSH_6mm, symbol Switch:SW_Push
- added U1: ESP32-S3-WROOM-1, RF_Module:ESP32-S3-WROOM-1, symbol RF_Module:ESP32-S3-WROOM-1
- added U6: AP2112K-3.3, Package_TO_SOT_SMD:SOT-23-5, symbol Regulator_Linear:AP2112K-3.3
- C1, C5: value 100nF -> 10uF
- C11: renamed from C12; value 1uF -> 2.2uF
- C16: renamed from C17; value 100nF -> 2.2uF
- C19: renamed from C20; value 1uF -> 4.7uF
- C22: value 10uF -> 1uF
- C3: value 100nF -> 1uF
- R11: renamed from R8; value 20k -> 10k
- R9: renamed from R6; value 20k -> 10k
- renumbered C11 to C10, C13 to C12, C14 to C13, C15 to C14, C16 to C15, C18 to C17, C19 to C18, C21 to C20, C7 to C6, C9 to C8, J4 to J3, R7 to R10, R9 to R12, R10 to R13, R11 to R14, R12 to R15, R13 to R16, R14 to R17, R16 to R18, R17 to R19, R21 to R20, R20 to R21, R18 to R22, R19 to R23, R2 to R5, R4 to R7, R5 to R8, PLAY/PAUSE1 to SW3, SW1 to SW4, BCKWRD/FRWD1 to SW5
Connections:
- net +3V3: now also J1.4 (VDD), R1.2, C7.1, C9.1, R2.1, R4.1, R6.1, U1.2 (3V3), U6.5 (VOUT); no longer BT1.2 (-), C10.1, C12.2, C15.2, C16.2, C19.1, C2.2, C20.1, C22.2, C3.1, C3.2, C4.2, C5.2, C6.2, C8.2, J1.6 (VSS), J1.SH (SHIELD), J2.S, J3.A1 (GND), J3.A12 (GND), J3.B1 (GND), J3.B12 (GND), J3.SH (SHIELD), R1.1, R12.1, R18.1, R22.1, R23.1, R7.2, SW3.1, SW4.C, SW4.S1, SW5.1, U2.10 (DEMP), U2.11 (FLT), U2.16 (FMT), U2.19 (DGND), U2.3 (CPGND), U2.9 (AGND), U3.2 (GND), U3.9 (GND), U4.1 (GND), U5.6 (V_{SS})
- net AMP_ENABLE: now also U1.10 (IO17)
- net BTN_NEXT: now also U1.9 (IO16)
- net BTN_PLAY: now also U1.11 (IO18)
- net DAC_MUTE: now also U1.22 (IO14)
- net ENC_A: now also U1.39 (IO1)
- net ENC_B: now also U1.38 (IO2)
- net GPIO10: now also R2.2, U1.18 (IO10)
- net GPIO11: now also R1.1, U1.19 (IO11)
- net GPIO12: now also U1.20 (IO12)
- net GPIO13: now also R3.1, U1.21 (IO13)
- net I2C_SCL: now also U1.12 (IO8)
- net I2C_SDA: now also U1.17 (IO9)
- net I2S_BCK: now also U1.5 (IO5)
- net I2S_DIN: now also U1.6 (IO6)
- net I2S_LRCK: now also U1.4 (IO4)
- net I2S_SCK: now also U1.7 (IO7)
- net USB_DN: now also J3.B7 (D-), U1.13 (USB_D-)
- net USB_DP: now also J3.B6 (D+), U1.14 (USB_D+)
- net VBAT: now also C21.2, U6.1 (VIN), U6.3 (EN)
- net GND: now reaches C1.2
- net GND: now also BT1.2 (-), C10.1, C12.2, C15.2, C16.2, C19.1, C2.2, C20.1, C22.2, C3.1, C4.2, C5.2, C6.2, C8.2, J1.6 (VSS), J1.SH (SHIELD), J2.S, J3.A1 (GND), J3.A12 (GND), J3.B1 (GND), J3.B12 (GND), J3.SH (SHIELD), R12.1, R18.1, R22.1, R23.1, R7.2, SW3.1, SW4.C, SW4.S1, SW5.1, U2.10 (DEMP), U2.11 (FLT), U2.16 (FMT), U2.19 (DGND), U2.3 (CPGND), U2.9 (AGND), U3.2 (GND), U3.9 (GND), U4.1 (GND), U5.6 (V_{SS}), C21.1, C7.2, C9.2, SW1.1, SW2.1, U1.1 (GND), U1.40 (GND), U1.41 (GND), U6.2 (GND); no longer J1.4 (VDD)
- net at J1.1 (DAT2): now also R6.2; no longer R1.2
- net ENC_BTN: now reaches R19.1, SW4.S2
- net ENC_BTN: now also U1.8 (IO15)
- net HP_DETECT: no longer names the net of J2.TN
- new net: C3.2, R4.2, SW1.2, U1.3 (EN)
- new net: SW2.2, U1.27 (IO0)
- no-connect marks 3 -> 2
Other:
- note added: "Battery (U5)"
- note added: "DAC (U2)"
- note added: "ESP32 (U1)"
- note added: "Headphone Jack (J2)"
- note added: "OLED (U4)"
- note added: "SD Card Module (J1)"
- note removed: "Battery (U4)"
- note removed: "DAC (U1)"
- note removed: "ESP32"
- note removed: "Headphone Jack"
- note removed: "OLED (U5)"
- note removed: "SD Card Module"
- title: (none) -> Fuji Mini
- moved on the sheet: C12, C17, C18, C6, C8, J1, J2, R10, R11, R12, R15, R16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

Commit message: Finished / Started the README / Added new gerbers
Parts:
- added TP1, TP2: GND, symbol Connector:TestPoint
- added TP3: +3V3, symbol Connector:TestPoint
- added TP4: VBAT, symbol Connector:TestPoint
- added TP5: VDD, symbol Connector:TestPoint
- added TP6: USB_DP, symbol Connector:TestPoint
- added TP7: USB_DN, symbol Connector:TestPoint
- C22: value 1uF -> 10uF
Connections:
- net +3V3: now also TP3.1
- net GND: now also TP1.1, TP2.1
- net USB_DN: now also TP7.1
- net USB_DP: now also TP6.1
- net VBAT: now also TP4.1
- net VDD: now also TP5.1
Other:
- moved on the sheet: J2

Commit message: Finishing up the designs / Fixing Issues / Trying new things
Parts:
- removed TP1, TP2: GND, symbol Connector:TestPoint
- removed TP3: +3V3, symbol Connector:TestPoint
- removed TP4: VBAT, symbol Connector:TestPoint
- removed TP5: VDD, symbol Connector:TestPoint
- removed TP6: USB_DP, symbol Connector:TestPoint
- removed TP7: USB_DN, symbol Connector:TestPoint
Connections:
- net +3V3: no longer D1.2 (A)
- net VBAT: now also D1.2 (A)

Commit message: New caps / fixing connections / new gerbers
Parts:
- C17, C18: footprint Capacitor_THT:CP_Radial_D6.3mm_P2.50mm -> Capacitor_SMD:CP_Elec_6.3x7.7
Changed lines of the file:
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@@
 			)
 		)
-		(property "Footprint" "Capacitor_THT:CP_Radial_D6.3mm_P2.50mm"
+		(property "Footprint" "Capacitor_SMD:CP_Elec_6.3x7.7"
 			(at 160.02 96.8248 0)
 			(hide yes)
@@
 			)
 		)
-		(property "Footprint" "Capacitor_THT:CP_Radial_D6.3mm_P2.50mm"
+		(property "Footprint" "Capacitor_SMD:CP_Elec_6.3x7.7"
 			(at 160.02 101.9048 0)
 			(hide yes)

Commit message: New gerbers, finished bom, new components
Parts:
- J1: footprint Connector_Card:microSD_HC_Hirose_DM3AT-SF-PEJM5 -> Connector_Card:microSD_HC_Molex_47219-2001
- J2: footprint Connector_Audio:Jack_3.5mm_CUI_SJ1-3535NG_Horizontal -> Connector_Audio:Jack_3.5mm_Lumberg_1503_02_Horizontal
Changed lines of the file:
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@@
 			)
 		)
-		(property "Footprint" "Connector_Audio:Jack_3.5mm_CUI_SJ1-3535NG_Horizontal"
+		(property "Footprint" "Connector_Audio:Jack_3.5mm_Lumberg_1503_02_Horizontal"
 			(at 186.69 99.06 0)
 			(hide yes)
@@
 			)
 		)
-		(property "Footprint" "Connector_Card:microSD_HC_Hirose_DM3AT-SF-PEJM5"
+		(property "Footprint" "Connector_Card:microSD_HC_Molex_47219-2001"
 			(at 96.52 152.4 0)
 			(hide yes)

Commit message: Finishing touches
Parts:
- removed U5: MCP73831-2-MC, Package_DFN_QFN:DFN-8-1EP_3x2mm_P0.5mm_EP1.7x1.4mm, symbol Battery_Management:MCP73831-2-MC
- added U5: MCP73831-2-OT, Package_TO_SOT_SMD:SOT-23-5, symbol Battery_Management:MCP73831-2-OT
Connections:
- net GND: now also U5.2 (V_{SS})
- net VBAT: now also U5.3 (V_{BAT})
- net VDD: now also U5.4 (V_{DD})
- net at R18.2: now also U5.5 (PROG)
- net at R20.1: now also U5.1 (STAT)
Changed lines of the file:
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@@
 	)
 	(symbol
+		(lib_id "Battery_Management:MCP73831-2-OT")
+		(at 215.9 151.13 0)
+		(unit 1)
+		(body_style 1)
+		(exclude_from_sim no)
+		(in_bom yes)
+		(on_board yes)
+		(in_pos_files yes)
+		(dnp no)
+		(property "Reference" "U5"
+			(at 215.138 150.622 0)
+			(show_name no)
+			(do_not_autoplace no)
+			(effects
+				(font
+					(size 0.635 0.635)
+				)
+				(justify left)
+			)
+		)
+		(property "Value" "MCP73831-2-OT"
+			(at 211.582 151.638 0)
+			(show_name no)
+			(do_not_autoplace no)
+			(effects
+				(font
+					(size 0.635 0.635)
+				)
+				(justify left)
+			)
+		)
+		(property "Footprint" "Package_TO_SOT_SMD:SOT-23-5"
+			(at 217.17 157.48 0)
+			(hide yes)
+			(show_name no)
+			(do_not_autoplace no)
+			(effects
+				(font
+					(size 1.27 1.27)
+					(italic yes)
+				)
+				(justify left)
+			)
+		)
+		(property "Datasheet" "http://ww1.microchip.com/downloads/en/DeviceDoc/20001984g.pdf"
+			(at 215.9 169.418 0)
+			(hide yes)
+			(show_name no)
+			(do_not_autoplace no)
+			(effects
+				(font
+					(size 1.27 1.27)
+				)
+			)
+		)
+		(property "Description" "Single cell, Li-Ion/Li-Po charge management controller, 4.20V, Tri-State Status Output, in SOT23-5 package"
+			(at 215.9 151.13 0)
+			(hide yes)
+			(show_name no)
+			(do_not_autoplace no)
+			(effects
+				(font
+					(size 1.27 1.27)
+				)
+			)
+		)
+		(pin "1"
+		)
+		(pin "5"
+		)
+		(pin "3"
+		)
+		(pin "2"
+		)
+		(pin "4"
+		)
+		(instances
+			(project "fuji-mini-v2"
+				(path "/cecf7a34-57e9-4b2e-844a-38f1c801dda5"
+					(reference "U5")
+					(unit 1)
+				)
+			)
+		)
+	)
+	(symbol
 		(lib_id "power:GND")
 		(at 110.49 180.34 0)
@@
 					(unit 1)
 				)
-			)
-		)
-	)
-	(symbol
-		(lib_id "Battery_Management:MCP73831-2-MC")
-		(at 215.9 151.13 0)
-		(unit 1)
-		(body_style 1)
-		(exclude_from_sim no)
-		(in_bom yes)
-		(on_board yes)
-		(in_pos_files yes)
-		(dnp no)
-		(property "Reference" "U5"
-			(at 212.09 149.352 0)
-			(show_name no)
-			(do_not_autoplace no)
-			(effects
-				(font
-					(size 0.635 0.635)
-				)
-				(justify left)
-			)
-		)
-		(property "Value" "MCP73831-2-MC"
-			(at 209.804 150.876 0)
-			(show_name no)
-			(do_not_autoplace no)
-			(effects
-				(font
-					(size 0.635 0.635)
-				)
-				(justify left)
-			)
-		)
-		(property "Footprint" "Package_DFN_QFN:DFN-8-1EP_3x2mm_P0.5mm_EP1.7x1.4mm"
-			(at 217.17 157.48 0)
-			(hide yes)
-			(show_name no)
-			(do_not_autoplace no)
-			(effects
-				(font
-					(size 1.27 1.27)
-					(italic yes)
-				)
-				(justify left)
-			)
-		)
-		(property "Datasheet" "http://ww1.microchip.com/downloads/en/DeviceDoc/20001984g.pdf"
-			(at 212.09 152.4 0)
-			(hide yes)
-			(show_name no)
-			(do_not_autoplace no)
-			(effects
-				(font
-					(size 1.27 1.27)
-				)
-			)
-		)
-		(property "Description" "Single cell, Li-Ion/Li-Po charge management controller, 4.20V, Tri-State Status Output, in DFN-8 package"
-			(at 215.9 151.13 0)
-			(hide yes)
-			(show_name no)
-			(do_not_autoplace no)
-			(effects
-				(font
-					(size 1.27 1.27)
-				)
-			)
-		)
-		(pin "4"
-		)
-		(pin "2"
-		)
-		(pin "6"
-		)
-		(pin "7"
-		)
-		(pin "8"
-		)
-		(pin "5"
-		)
-		(pin "3"
-		)
-		(pin "1"
-		)
-		(instances
-			(project "fuji-mini-v2"
-				(path "/cecf7a34-57e9-4b2e-844a-38f1c801dda5"
-					(reference "U5")
-					(unit 1)
-				)
