File: fuji-mini-v2/_autosave-fuji-mini-v2.kicad_sch (KiCad schematic)
At the start: 58 parts, among them J1 Micro_SD_Card, J2 AudioJack3_SwitchT, J4 USB_C_Receptacle_USB2.0_14P, SW1 RotaryEncoder_Switch, U1 ESP32-S3, U2 PCM5102A, U3 TPA6110A2DGN, U4 ER_OLEDM0.91_1x-I2C, U5 MCP73831-2-MC, U6 AMS1117-3.3

Commit message: Footprints + PCB v1.0
Parts:
- J4: footprint (none) -> Connector_USB:USB_C_Receptacle_XKB_U262-16XN-4BVC11
Changed lines of the file:
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@@
 			)
 		)
-		(property "Footprint" ""
+		(property "Footprint" "Connector_USB:USB_C_Receptacle_XKB_U262-16XN-4BVC11"
 			(at 246.38 106.68 0)
 			(hide yes)
