File: fuji-mini-v2/fuji-mini-v2.kicad_pcb (KiCad board)
At the start: 2 copper layers, 58.4 x 81.3 mm, 58 parts, among them J1 Micro_SD_Card, J2 AudioJack3_SwitchT, J4 USB_C_Receptacle_USB2.0_14P, SW1 RotaryEncoder_Switch, U1 ESP32-S3, U2 PCM5102A, U3 TPA6110A2DGN, U4 ER_OLEDM0.91_1x-I2C, U5 MCP73831-2-MC, U6 AMS1117-3.3

Commit message: made the edge cut wider
Parts:
- added G***: LOGO, LOGO, F.Cu at (83.8, 59.4)
Routing:
- net Net-(D1-K): track 67.1 -> 119.7 mm
- net Net-(U2-VNEG): track 103.5 -> 151.2 mm
- net 3V3: track 654.1 -> 685.5 mm
- net Net-(U2-CAPM): track 92.0 -> 103.9 mm
- net I2C_SDA: track 59.9 -> 49.4 mm
- net Net-(R17-Pad1): track 19.2 -> 22.6 mm
- net I2S_LRCK: track 113.1 -> 115.4 mm
- net HP_R: track 16.0 -> 17.5 mm
- net HP_L: track 22.4 -> 23.4 mm
Other:
- board text added: "Fuji Mini"
- board text added: "Made by A41K"
