File: fuji-mini-v2/fuji-mini-v2.kicad_pcb (KiCad board)
At the start: 2 copper layers, 73.8 x 97.7 mm, 64 parts, among them J1 Micro_SD_Card, J2 AudioJack3_SwitchT, J3 USB_C_Receptacle_USB2.0_14P, SW1 SW_Push, SW2 SW_Push, SW3 SW_Push, SW4 RotaryEncoder_Switch, SW5 SW_Push, U1 ESP32-S3-WROOM-1, U2 PCM5102A, U3 TPA6110A2DGN, U4 ER_OLEDM0.91_1x-I2C, U5 MCP73831-2-MC, U6 AP2112K-3.3

Commit message: New caps / fixing connections / new gerbers
Parts:
- C17, C18: footprint Capacitor_THT:CP_Radial_D6.3mm_P2.50mm -> Capacitor_SMD:CP_Elec_6.3x7.7
- moved C17 2.50 mm to (134.6, 137.2), turned to 90 degrees
- moved C18 1.82 mm to (127.0, 137.2), turned to 90 degrees
Routing:
- net HP_R: track 28.2 -> 37.0 mm, vias 0 -> 2
- net I2C_SCL: track 204.8 -> 198.4 mm
- net HP_L: track 13.6 -> 17.9 mm
- net +3V3: track 341.6 -> 344.9 mm
- net I2S_DIN: track 89.3 -> 85.9 mm
- net VO1: track 42.5 -> 45.6 mm, vias 3 -> 4
- net USB_DN: track 86.0 -> 87.8 mm
- net VO2: track 50.1 -> 51.5 mm
- net ENC_A: track 120.5 -> 121.8 mm

Commit message: New gerbers, finished bom, new components
Parts:
- J1: footprint Connector_Card:microSD_HC_Hirose_DM3AT-SF-PEJM5 -> Connector_Card:microSD_HC_Molex_47219-2001
- J2: footprint Connector_Audio:Jack_3.5mm_CUI_SJ1-3535NG_Horizontal -> Connector_Audio:Jack_3.5mm_Lumberg_1503_02_Horizontal
- U5: value MCP73831-2-MC -> MCP73831-2-OT; footprint Package_DFN_QFN:DFN-8-1EP_3x2mm_P0.5mm_EP1.7x1.4mm -> Package_TO_SOT_SMD:SOT-23-5
- moved J1 6.18 mm to (141.0, 102.2), turned to -90 degrees
- moved J2 1.86 mm to (143.6, 144.8)
- moved U5 0.56 mm to (80.6, 87.0)
Connections:
- U5 pad 1: VDD -> Net-(U5-STAT)
- U5 pad 2: VDD -> GND
- U5 pad 4: VBAT -> VDD
- U5 pad 5: Net-(U5-STAT) -> Net-(U5-PROG)
Routing:
- net GND: track 603.1 -> 628.5 mm, vias 16 -> 15
- net HP_L: track 17.9 -> 40.2 mm
- net GPIO12: track 43.3 -> 61.8 mm
- net GPIO13: track 81.5 -> 98.2 mm
- net GPIO10: track 45.7 -> 62.4 mm, vias 4 -> 5
- net Net-(J1-DAT1): track 10.8 -> 27.3 mm
- net GPIO11: track 49.4 -> 65.9 mm
- net +3V3: track 344.9 -> 360.9 mm
- net Net-(U5-STAT): track 20.1 -> 31.0 mm
- net HP_R: track 37.0 -> 29.3 mm
- net Net-(J1-DAT2): track 38.1 -> 44.4 mm
- net VDD: track 83.9 -> 89.2 mm
- net VBAT: track 215.5 -> 213.5 mm
- net Net-(U3-IN2-): track 34.7 -> 33.8 mm
- net Net-(U5-PROG): track 9.44 -> 8.94 mm
